Commit message: kyle's robot changes

File: my_robot_description/urdf/arm.xacro (robot description, xacro)
@@ -15,5 +15,5 @@
     <xacro:property name = "eef_left_length" value = ".02" />
     <xacro:property name = "eef_left_width" value = ".02" />
-    <xacro:property name = "eef_left_height" value = ".30" />
+    <xacro:property name = "eef_left_height" value = ".25" />
     <xacro:property name = "eef_right_length" value = ".02" />
     <xacro:property name = "eef_right_width" value = ".02" />
@@ -59,5 +59,5 @@
             <origin xyz = "0 0 ${forearm_length/2}" rpy="0 0 0" />
         </collision>
-        <xacro:wheel_inertia m = ".3" r = "${forearm_radius}" l = "${forearm_length}"
+        <xacro:wheel_inertia m = ".1" r = "${forearm_radius}" l = "${forearm_length}"
                                 o_xyz="0 0 ${forearm_length/2}" o_rpy="0 0 0"/>
     </link>
@@ -75,5 +75,5 @@
                 <cylinder radius="${hand_radius}" length = "${hand_length}" />
             </geometry>
-            <origin xyz = "0 0 ${hand_length/2}" rpy="0 0 0" />
+            <origin xyz = "0 ${forearm_radius*2} ${hand_length/2}" rpy="0 0 0" />
             <material name="orange"/>
         </visual>
@@ -82,8 +82,8 @@
                 <cylinder radius="${hand_radius}" length = "${hand_length}" />
             </geometry>
-            <origin xyz = "0 0 ${hand_length/2}" rpy="0 0 0" />
+            <origin xyz = "0 ${forearm_radius*2} ${hand_length/2}" rpy="0 0 0" />
         </collision>
-        <xacro:wheel_inertia m = ".3" r = "${hand_radius}" l = "${hand_length}"
-                                o_xyz="0 0 ${hand_length/2}" o_rpy="0 0 0"/>
+        <xacro:wheel_inertia m = ".1" r = "${hand_radius}" l = "${hand_length}"
+                                o_xyz="0 ${forearm_radius*2} ${hand_length/2}" o_rpy="0 0 0"/>
     </link>
     <joint name="forearm_hand_joint" type = "revolute">
@@ -109,5 +109,5 @@
             <origin xyz = "0 0 ${hand_2_length/2}" rpy="0 0 0" />
         </collision>
-        <xacro:wheel_inertia m = ".3" r = "${hand_2_radius}" l = "${hand_2_length}"
+        <xacro:wheel_inertia m = ".1" r = "${hand_2_radius}" l = "${hand_2_length}"
                                 o_xyz="0 0 ${hand_2_length/2}" o_rpy="0 0 0"/>
     </link>
@@ -125,5 +125,5 @@
                 <box size="${eef_length} ${eef_width} ${eef_height}"/>
             </geometry>
-            <origin xyz = "0 0 0" rpy="0 0 0" />
+            <origin xyz = "0 0 ${eef_length/2}" rpy="0 0 0" />
             <material name="blue"/>
         </visual>
@@ -132,8 +132,8 @@
                 <box size="${eef_length} ${eef_width} ${eef_height}"/>
             </geometry>
-            <origin xyz = "0 0 0" rpy="0 0 0" />
+            <origin xyz = "0 0 ${eef_length/2}" rpy="0 0 0" />
         </collision>
-        <xacro:box_inertia m = ".3" x = "${eef_length}" y = "${eef_width}" z = "${eef_height}"
-                            o_xyz="0 0 0" o_rpy="0 0 0"/>
+        <xacro:box_inertia m = ".01" x = "${eef_length}" y = "${eef_width}" z = "${eef_height}"
+                            o_xyz="0 0 ${eef_length/2}" o_rpy="0 0 0"/>
     </link>
     <joint name="hand_2_eef_joint" type = "fixed">
@@ -148,5 +148,5 @@
                 <box size="${eef_left_length} ${eef_left_width} ${eef_left_height}"/>
             </geometry>
-            <origin xyz = "0 0 ${eef_left_height/2}" rpy="0 0 0" />
+            <origin xyz = "${eef_right_width} 0 ${eef_left_height/2}" rpy="0 0 0" />
             <material name="blue"/>
         </visual>
@@ -155,8 +155,8 @@
                 <box size="${eef_left_length} ${eef_left_width} ${eef_left_height}"/>
             </geometry>
-            <origin xyz = "0 0 ${eef_left_height}" rpy="0 0 0" />
+            <origin xyz = "${eef_right_width} 0 ${eef_left_height/2}" rpy="0 0 0" />
         </collision>
-        <xacro:box_inertia m = ".3" x = "${eef_left_length}" y = "${eef_left_width}" z = "${eef_left_height}"
-                            o_xyz="0 0 0" o_rpy="0 0 0"/>
+        <xacro:box_inertia m = ".01" x = "${eef_left_length}" y = "${eef_left_width}" z = "${eef_left_height}"
+                            o_xyz="${eef_right_width} 0 ${eef_left_height/2}" o_rpy="0 0 0"/>
     </link>
     <joint name="eef_eef_left_joint" type = "revolute">
@@ -173,5 +173,5 @@
                 <box size="${eef_right_length} ${eef_right_width} ${eef_right_height}"/>
             </geometry>
-            <origin xyz = "0 0 0" rpy="0 0 0" />
+            <origin xyz = "${eef_right_width} 0 0" rpy="0 0 0" />
             <material name="blue"/>
         </visual>
@@ -180,8 +180,8 @@
                 <box size="${eef_right_length} ${eef_right_width} ${eef_right_height}"/>
             </geometry>
-            <origin xyz = "0 0 0" rpy="0 0 0" />
+            <origin xyz = "${eef_right_width} 0 0" rpy="0 0 0" />
         </collision>
-        <xacro:box_inertia m = ".3" x = "${eef_right_length}" y = "${eef_right_width}" z = "${eef_right_height}"
-                            o_xyz="0 0 0" o_rpy="0 0 0"/>
+        <xacro:box_inertia m = ".01" x = "${eef_right_length}" y = "${eef_right_width}" z = "${eef_right_height}"
+                            o_xyz="${eef_right_width} 0 0" o_rpy="0 0 0"/>
     </link>
     <joint name="eef_eef_right_joint" type = "fixed">

File: my_robot_description/urdf/camera.xacro (robot description, xacro)
@@ -11,16 +11,28 @@
             <material name="grey" />
         </visual>
-        <collision>
+        <!-- <collision>
             <geometry>
                 <box size="${camera_length} ${camera_width} ${camera_height}" />
             </geometry>
         </collision>
-        <xacro:box_inertia m="0.1" x="${camera_length}" y="${camera_width}" z="${camera_height}"
-                           o_xyz="0 0 0" o_rpy="0 0 0" />
+        <xacro:box_inertia m="0.001" x="${camera_length}" y="${camera_width}" z="${camera_height}"
+                           o_xyz="0 0 0" o_rpy="0 0 0" /> -->
     </link>
-    <joint name="base_camera_joint" type="fixed">
+    <!-- <joint name="base_camera_joint" type="fixed">
         <parent link="hand_2_link" />
         <child link="camera_link" />
-        <origin xyz="${-hand_2_radius} 0 ${hand_2_length}" rpy="0 ${-pi/2} 0" />
+        <origin xyz="${-hand_2_radius*2} 0 ${hand_2_length}" rpy="0 ${-pi/2} 0" />
+    </joint>
+    <link name="camera_link_optical" />
+    <joint name="camera_optical_joint" type="fixed">
+        <origin xyz="0 0 0" rpy="${-pi/2} 0 ${-pi/2}"/>
+        <parent link="camera_link"/>
+        <child link="camera_link_optical"/>
+    </joint> -->
+    <!-- Move camera to front of TARo for debugging -->
+    <joint name="base_camera_joint" type="fixed">
+        <parent link="base_link" />
+        <child link="camera_link" />
+        <origin xyz="${base_length/2+camera_length/2} 0 ${base_height/2}" rpy="0 0 0" />
     </joint>
     <link name="camera_link_optical" />
@@ -30,4 +42,5 @@
         <child link="camera_link_optical"/>
     </joint>
+    <!-- Move camera to front of TARo for debugging -->
     <gazebo reference="camera_link">
         <sensor name="camera" type="camera">
@@ -40,6 +53,6 @@
                 </image>
                 <clip>
-                    <near>0.1</near>
-                    <far>15</far>
+                    <near>0.005</near>
+                    <far>20.0</far>
                 </clip>
                 <noise>
@@ -52,5 +65,5 @@
             </camera>
             <always_on>1</always_on>
-            <update_rate>20</update_rate>
+            <update_rate>60</update_rate>
             <visualize>true</visualize>
             <topic>camera/image_raw</topic>

File: my_robot_description/urdf/mobile_base.xacro (robot description, xacro)
@@ -6,21 +6,125 @@
     <xacro:property name = "wheel_radius" value = ".2" />
     <xacro:property name = "wheel_length" value = ".1" />
+    <xacro:property name = "base_length_h" value = ".6" />
+    <xacro:property name = "base_thickness" value = ".01" />
     <link name="base_footprint"/>
     <link name="base_link">
         <visual>
             <geometry>
-                <box size="${base_length} ${base_width} ${base_height}"/>
-            </geometry>
-            <origin xyz = "0 0 ${base_height/2}" rpy="0 0 0" />
-            <material name="blue"/>
-        </visual>
-        <collision>
-            <geometry>
-                <box size="${base_length} ${base_width} ${base_height}"/>
-            </geometry>
-            <origin xyz = "0 0 ${base_height/2}" rpy="0 0 0" />
-        </collision>
-        <xacro:box_inertia m = "5.0" x = "${base_length}" y = "${base_width}" z = "${base_height}"
-                            o_xyz="0 0 ${base_height/2}" o_rpy="0 0 0"/>
+                <box size="${base_length_h} ${base_width} ${base_height}"/>
+            </geometry>
+            <origin xyz = "${base_length_h/2} 0 ${base_height/2}" rpy="0 0 0" />
+            <material name="blue"/>
+        </visual>
+        <collision>
+            <geometry>
+                <box size="${base_length_h} ${base_width} ${base_height}"/>
+            </geometry>
+            <origin xyz = "${base_length_h/2} 0 ${base_height/2}" rpy="0 0 0" />
+        </collision>
+        <xacro:box_inertia m = "5.0" x = "${base_length_h}" y = "${base_width}" z = "${base_height}"
+                            o_xyz="${base_length_h/2} 0 ${base_height/2}" o_rpy="0 0 0"/>
+    </link>
+    <link name="base_link_floor">
+        <visual>
+            <geometry>
+                <box size="${base_length_h} ${base_width-2*base_thickness} ${base_thickness}"/>
+            </geometry>
+            <origin xyz = "${-base_length_h/2} 0 ${base_thickness/2}" rpy="0 0 0" />
+            <material name="grey"/>
+        </visual>
+        <collision>
+            <geometry>
+                <box size="${base_length_h} ${base_width-2*base_thickness} ${base_thickness}"/>
+            </geometry>
+            <origin xyz = "${-base_length_h/2} 0 ${base_thickness/2}" rpy="0 0 0" />
+        </collision>
+        <xacro:box_inertia m = "2" x = "${base_length_h}" y = "${base_width-2*base_thickness}" z = "${base_thickness}"
+                            o_xyz="${-base_length_h/2} 0 ${base_thickness/2}" o_rpy="0 0 0"/>
+    </link>
+    <link name="base_link_wall_left">
+        <visual>
+            <geometry>
+                <box size="${base_length_h} ${base_thickness} ${base_height}"/>
+            </geometry>
+            <origin xyz = "${-base_length_h/2} ${base_width/2-base_thickness/2} ${base_height/2}" rpy="0 0 0" />
+            <material name="blue"/>
+        </visual>
+        <collision>
+            <geometry>
+                <box size="${base_length_h} ${base_thickness} ${base_height}"/>
+            </geometry>
+            <origin xyz = "${-base_length_h/2} ${base_width/2-base_thickness/2} ${base_height/2}" rpy="0 0 0" />
+        </collision>
+        <xacro:box_inertia m = "2" x = "${base_length_h}" y = "${base_thickness}" z = "${base_height}"
+                            o_xyz="${-base_length_h/2} ${base_width/2-base_thickness/2} ${base_height/2}" o_rpy="0 0 0"/>
+    </link>
+    <link name="base_link_wall_right">
+        <visual>
+            <geometry>
+                <box size="${base_length_h} ${base_thickness} ${base_height}"/>
+            </geometry>
+            <origin xyz = "${-base_length_h/2} -${base_width/2-base_thickness/2} ${base_height/2}" rpy="0 0 0" />
+            <material name="blue"/>
+        </visual>
+        <collision>
+            <geometry>
+                <box size="${base_length_h} ${base_thickness} ${base_height}"/>
+            </geometry>
+            <origin xyz = "${-base_length_h/2} -${base_width/2-base_thickness/2} ${base_height/2}" rpy="0 0 0" />
+        </collision>
+        <xacro:box_inertia m = "2" x = "${base_length_h}" y = "${base_thickness}" z = "${base_height}"
+                            o_xyz="${-base_length_h/2} -${base_width/2-base_thickness/2} ${base_height/2}" o_rpy="0 0 0"/>
+    </link>
+    <link name="base_link_wall_rear_mid">
+        <visual>
+            <geometry>
+                <box size="${base_thickness} ${base_width-base_thickness*2} ${base_height}"/>
+            </geometry>
+            <origin xyz = "-${base_length_h/2+base_thickness} 0 ${base_height/2}" rpy="0 0 0" />
+            <material name="grey"/>
+        </visual>
+        <collision>
+            <geometry>
+                <box size="${base_thickness} ${base_width-base_thickness*2} ${base_height}"/>
+            </geometry>
+            <origin xyz = "-${base_length_h/2+base_thickness} 0 ${base_height/2}" rpy="0 0 0" />
+        </collision>
+        <xacro:box_inertia m = "2" x = "${base_thickness}" y = "${base_width-base_thickness*2}" z = "${base_height}"
+                            o_xyz="-${base_length_h/2+base_thickness} 0 ${base_height/2}" o_rpy="0 0 0"/>
+    </link>
+    <link name="base_link_wall_rear_end">
+        <visual>
+            <geometry>
+                <box size="${base_thickness} ${base_width} ${base_height}"/>
+            </geometry>
+            <origin xyz = "-${base_length_h} 0 ${base_height/2}" rpy="0 0 0" />
+            <material name="blue"/>
+        </visual>
+        <collision>
+            <geometry>
+                <box size="${base_thickness} ${base_width} ${base_height}"/>
+            </geometry>
+            <origin xyz = "-${base_length_h} 0 ${base_height/2}" rpy="0 0 0" />
+        </collision>
+        <xacro:box_inertia m = "2" x = "${base_thickness}" y = "${base_width}" z = "${base_height}"
+                            o_xyz="-${base_length_h} 0 ${base_height/2}" o_rpy="0 0 0"/>
+    </link>
+    <link name="base_link_wall_split">
+        <visual>
+            <geometry>
+                <box size="${base_length_h} ${base_thickness} ${base_height}"/>
+            </geometry>
+            <origin xyz = "${-base_length_h/2} 0 ${base_height/2}" rpy="0 0 0" />
+            <material name="grey"/>
+        </visual>
+        <collision>
+            <geometry>
+                <box size="${base_length_h} ${base_thickness} ${base_height}"/>
+            </geometry>
+            <origin xyz = "${-base_length_h/2} 0 ${base_height/2}" rpy="0 0 0" />
+        </collision>
+        <xacro:box_inertia m = "2" x = "${base_length_h}" y = "${base_thickness}" z = "${base_height}"
+                            o_xyz="${-base_length_h/2} 0 ${base_height/2}" o_rpy="0 0 0"/>
     </link>
     <xacro:macro name = "wheel_link" params="prefix">
@@ -63,5 +167,35 @@
     <joint name="base_joint" type="fixed">
         <parent link = "base_footprint"/>
+        <child link="base_link_floor"/>
+        <origin xyz = "0 0 ${wheel_radius}" rpy = "0 0 0"/>
+    </joint>
+    <joint name="base_joint_floor" type="fixed">
+        <parent link = "base_footprint"/>
         <child link="base_link"/>
+        <origin xyz = "0 0 ${wheel_radius}" rpy = "0 0 0"/>
+    </joint>
+    <joint name="base_joint_left_wall" type="fixed">
+        <parent link = "base_footprint"/>
+        <child link="base_link_wall_left"/>
+        <origin xyz = "0 0 ${wheel_radius}" rpy = "0 0 0"/>
+    </joint>
+    <joint name="base_joint_right_wall" type="fixed">
+        <parent link = "base_footprint"/>
+        <child link="base_link_wall_right"/>
+        <origin xyz = "0 0 ${wheel_radius}" rpy = "0 0 0"/>
+    </joint>
+    <joint name="base_joint_rear_wall_mid" type="fixed">
+        <parent link = "base_footprint"/>
+        <child link="base_link_wall_rear_mid"/>
+        <origin xyz = "0 0 ${wheel_radius}" rpy = "0 0 0"/>
+    </joint>
+    <joint name="base_joint_rear_wall_end" type="fixed">
+        <parent link = "base_footprint"/>
+        <child link="base_link_wall_rear_end"/>
+        <origin xyz = "0 0 ${wheel_radius}" rpy = "0 0 0"/>
+    </joint>
+    <joint name="base_joint_rear_wall_split" type="fixed">
+        <parent link = "base_footprint"/>
+        <child link="base_link_wall_split"/>
         <origin xyz = "0 0 ${wheel_radius}" rpy = "0 0 0"/>
     </joint>
