Commit message: yolo and arm comms ok
(cherry picked from commit 15fecc686a5b487c8f431aec169e144fa19316a7)

init change for robotics tool box

current_stuff

yay detects_waste bad bounding box

messed up seeting to initial

fix bad transition

move camera back to arm

we are yolo ing again

File: my_robot_description/urdf/camera.xacro (robot description, xacro)
@@ -19,5 +19,5 @@
                            o_xyz="0 0 0" o_rpy="0 0 0" /> -->
     </link>
-    <!-- <joint name="base_camera_joint" type="fixed">
+    <joint name="base_camera_joint" type="fixed">
         <parent link="hand_2_link" />
         <child link="camera_link" />
@@ -29,7 +29,7 @@
         <parent link="camera_link"/>
         <child link="camera_link_optical"/>
-    </joint> -->
+    </joint>
     <!-- Move camera to front of TARo for debugging -->
-    <joint name="base_camera_joint" type="fixed">
+    <!-- <joint name="base_camera_joint" type="fixed">
         <parent link="base_link" />
         <child link="camera_link" />
@@ -41,5 +41,5 @@
         <parent link="camera_link"/>
         <child link="camera_link_optical"/>
-    </joint>
+    </joint> -->
     <!-- Move camera to front of TARo for debugging -->
     <gazebo reference="camera_link">

Commit message: move camera in eef

File: my_robot_description/urdf/camera.xacro (robot description, xacro)
@@ -22,5 +22,5 @@
         <parent link="hand_2_link" />
         <child link="camera_link" />
-        <origin xyz="${-hand_2_radius*2} 0 ${hand_2_length}" rpy="0 ${-pi/2} 0" />
+        <origin xyz="${hand_2_radius*0.5} 0 ${hand_2_length}" rpy="0 ${-pi/2} 0" />
     </joint>
     <link name="camera_link_optical" />
